File: 16ChannelServoControllerDaughterboardDesign.kicad_pcb (KiCad board)
At the start: 2 copper layers, 100 x 53.5 mm, 19 parts, among them J1 DaughterBoard, J2 8ServoConnectSym, J3 8ServoConnectSym, J4 Conn_01x03, J6 Screw_Terminal_01x02, Q1 BSS138, Q2 BSS138, U1 PCA9685PW

Commit message: updated some things
Parts:
- J6: footprint TerminalBlock:TerminalBlock_Altech_AK300-2_P5.00mm -> TerminalBlock_Phoenix:TerminalBlock_Phoenix_MKDS-1,5-2_1x02_P5.00mm_Horizontal
- moved J6 5.57 mm to (117.1, 78.6), turned to 180 degrees
Connections:
- J6 pad 1: GND -> +6V
- J6 pad 2: +6V -> GND
