File: 16ChannelServoControllerDaughterboardDesign.kicad_sch (KiCad schematic)
At the start: 18 parts, among them J1 DaughterBoard, J2 8ServoConnectSym, J3 8ServoConnectSym, J4 Conn_01x03, J6 Screw_Terminal_01x02, Q1 BSS138, Q2 BSS138, U1 PCA9685PW

Commit message: updated some things
Parts:
- J6: footprint TerminalBlock:TerminalBlock_Altech_AK300-2_P5.00mm -> TerminalBlock_Phoenix:TerminalBlock_Phoenix_MKDS-1,5-2_1x02_P5.00mm_Horizontal
Connections:
- net +6V: now also J6.1 (Pin_1); no longer J6.2 (Pin_2)
- net GND: now also J6.2 (Pin_2); no longer J6.1 (Pin_1)
Other:
- moved on the sheet: J6
Changed lines of the file:
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@@
 (kicad_sch
-	(version 20231120)
+	(version 20250114)
 	(generator "eeschema")
-	(generator_version "8.0")
+	(generator_version "9.0")
 	(paper "A4")
+	(rectangle
+		(start 12.7 125.73)
+		(end 81.28 196.85)
+		(stroke
+			(width 1.016)
+			(type default)
+		)
+		(fill
+			(type none)
+		)
+	)
+	(rectangle
+		(start 160.02 12.7)
+		(end 199.39 57.15)
+		(stroke
+			(width 1.016)
+			(type default)
+		)
+		(fill
+			(type none)
+		)
+	)
+	(rectangle
+		(start 12.7 64.77)
+		(end 81.28 125.73)
+		(stroke
+			(width 1.016)
+			(type default)
+		)
+		(fill
+			(type none)
+		)
+	)
+	(rectangle
+		(start 81.28 12.7)
+		(end 160.02 101.6)
+		(stroke
+			(width 1.016)
+			(type default)
+		)
+		(fill
+			(type none)
+		)
+	)
+	(rectangle
+		(start 81.28 101.6)
+		(end 160.02 196.85)
+		(stroke
+			(width 1.016)
+			(type default)
+		)
+		(fill
+			(type none)
+		)
+	)
+	(rectangle
+		(start 12.7 12.7)
+		(end 81.28 64.77)
+		(stroke
+			(width 1.016)
+			(type default)
+		)
+		(fill
+			(type none)
+		)
+	)
+	(text "Bidirectional voltage translator \n+3V3 <-> +5V for I2C pins (SDA & SCL)"
+		(exclude_from_sim no)
+		(at 14.986 68.834 0)
+		(effects
+			(font
+				(size 1.651 1.651)
+				(thickness 0.254)
+				(bold yes)
+			)
+			(justify left)
+		)
+	)
+	(text "Servo connectors \n(16 sets of three pin servo connectors)"
+		(exclude_from_sim no)
+		(at 13.716 130.302 0)
+		(effects
+			(font
+				(size 1.651 1.651)
+				(thickness 0.254)
+				(bold yes)
+			)
+			(justify left)
+		)
+	)
+	(text "Daughterboard"
+		(exclude_from_sim no)
+		(at 83.312 106.426 0)
+		(effects
+			(font
+				(size 1.651 1.651)
+				(thickness 0.254)
+				(bold yes)
+			)
+			(justify left)
+		)
+	)
+	(text "Power flags"
+		(exclude_from_sim no)
+		(at 161.29 16.002 0)
+		(effects
+			(font
+				(size 1.651 1.651)
+				(thickness 0.254)
+				(bold yes)
+			)
+			(justify left)
+		)
+	)
+	(text "Servo power in (+6V)"
+		(exclude_from_sim no)
+		(at 14.732 15.748 0)
+		(effects
+			(font
+				(size 1.651 1.651)
+				(thickness 0.254)
+				(bold yes)
+			)
+			(justify left)
+		)
+	)
+	(text "PCA9685 & decoupling capacitor (place close to VCC pin)"
+		(exclude_from_sim no)
+		(at 82.296 16.256 0)
+		(effects
+			(font
+				(size 1.651 1.651)
+				(thickness 0.254)
+				(bold yes)
+			)
+			(justify left)
+		)
+	)
 	(junction
 		(at 54.61 30.48)
@@
 		)
 	)
-	(rectangle
-		(start 12.7 125.73)
-		(end 81.28 196.85)
-		(stroke
-			(width 1.016)
-			(type default)
-		)
-		(fill
-			(type none)
-		)
-	)
-	(rectangle
-		(start 160.02 12.7)
-		(end 199.39 57.15)
-		(stroke
-			(width 1.016)
-			(type default)
-		)
-		(fill
-			(type none)
-		)
-	)
-	(rectangle
-		(start 12.7 64.77)
-		(end 81.28 125.73)
-		(stroke
-			(width 1.016)
-			(type default)
-		)
-		(fill
-			(type none)
-		)
-	)
-	(rectangle
-		(start 81.28 12.7)
-		(end 160.02 101.6)
-		(stroke
-			(width 1.016)
-			(type default)
-		)
-		(fill
-			(type none)
-		)
-	)
-	(rectangle
-		(start 81.28 101.6)
-		(end 160.02 196.85)
-		(stroke
-			(width 1.016)
-			(type default)
-		)
-		(fill
-			(type none)
-		)
-	)
-	(rectangle
-		(start 12.7 12.7)
-		(end 81.28 64.77)
-		(stroke
-			(width 1.016)
-			(type default)
-		)
-		(fill
-			(type none)
-		)
-	)
-	(text "Bidirectional voltage translator \n+3V3 <-> +5V for I2C pins (SDA & SCL)"
-		(exclude_from_sim no)
-		(at 14.986 68.834 0)
-		(effects
-			(font
-				(size 1.651 1.651)
-				(thickness 0.254)
-				(bold yes)
-			)
-			(justify left)
-		)
-	)
-	(text "Servo connectors \n(16 sets of three pin servo connectors)"
-		(exclude_from_sim no)
-		(at 13.716 130.302 0)
-		(effects
-			(font
-				(size 1.651 1.651)
-				(thickness 0.254)
-				(bold yes)
-			)
-			(justify left)
-		)
-	)
-	(text "Daughterboard"
-		(exclude_from_sim no)
-		(at 83.312 106.426 0)
-		(effects
-			(font
-				(size 1.651 1.651)
-				(thickness 0.254)
-				(bold yes)
-			)
-			(justify left)
-		)
-	)
-	(text "Power flags"
-		(exclude_from_sim no)
-		(at 161.29 16.002 0)
-		(effects
-			(font
-				(size 1.651 1.651)
-				(thickness 0.254)
-				(bold yes)
-			)
-			(justify left)
-		)
-	)
-	(text "Servo power in (+6V)"
-		(exclude_from_sim no)
-		(at 14.732 15.748 0)
-		(effects
-			(font
-				(size 1.651 1.651)
-				(thickness 0.254)
-				(bold yes)
-			)
-			(justify left)
-		)
-	)
-	(text "PCA9685 & decoupling capacitor (place close to VCC pin)"
-		(exclude_from_sim no)
-		(at 82.296 16.256 0)
-		(effects
-			(font
-				(size 1.651 1.651)
-				(thickness 0.254)
-				(bold yes)
-			)
-			(justify left)
-		)
-	)
 	(global_label "SDA_3V3"
 		(shape bidirectional)
@@
 			)
 		)
-		(property "Description" ""
+		(property "Description" "Light emitting diode"
+			(at 45.72 48.26 0)
+			(effects
+				(font
+					(size 1.27 1.27)
+				)
+				(hide yes)
+			)
+		)
+		(property "Sim.Pins" "1=K 2=A"
 			(at 45.72 48.26 0)
 			(effects
@@
 	)
 	(symbol
-		(lib_name "VCC_2")
 		(lib_id "power:VCC")
 		(at 45.72 26.67 0)
@@
 			)
 		)
-		(property "Description" ""
+		(property "Description" "Resistor, US symbol"
 			(at 45.72 38.1 0)
 			(effects
@@
 	)
 	(symbol
-		(lib_name "VCC_2")
 		(lib_id "power:VCC")
 		(at 184.15 36.83 0)
@@
 			)
 		)
-		(property "Description" ""
+		(property "Description" "Polarized capacitor"
 			(at 54.61 44.45 0)
 			(effects
@@
 	(symbol
 		(lib_id "Connector:Screw_Terminal_01x02")
-		(at 25.4 33.02 180)
+		(at 25.4 30.48 0)
+		(mirror y)
 		(unit 1)
 		(exclude_from_sim no)
@@
 		(on_board yes)
 		(dnp no)
-		(fields_autoplaced yes)
 		(property "Reference" "J6"
-			(at 25.4 24.638 0)
+			(at 25.4 38.862 0)
 			(effects
 				(font
@@
 		)
 		(property "Value" "Screw_Terminal_01x02"
-			(at 25.4 27.178 0)
+			(at 25.4 36.322 0)
 			(effects
 				(font
@@
 			)
 		)
-		(property "Footprint" "TerminalBlock:TerminalBlock_Altech_AK300-2_P5.00mm"
-			(at 25.4 33.02 0)
+		(property "Footprint" "TerminalBlock_Phoenix:TerminalBlock_Phoenix_MKDS-1,5-2_1x02_P5.00mm_Horizontal"
+			(at 25.4 30.48 0)
 			(effects
 				(font
@@
 		)
 		(property "Datasheet" "~"
-			(at 25.4 33.02 0)
+			(at 25.4 30.48 0)
 			(effects
 				(font
@@
 			)
 		)
-		(property "Description" ""
-			(at 25.4 33.02 0)
+		(property "Description" "Generic screw terminal, single row, 01x02, script generated (kicad-library-utils/schlib/autogen/connector/)"
+			(at 25.4 30.48 0)
 			(effects
 				(font
@@
 			)
 		)
-		(property "Description" ""
+		(property "Description" "Unpolarized capacitor"
 			(at 90.17 85.09 0)
 			(effects
@@
 			)
 		)
-		(property "Description" ""
+		(property "Description" "Unpolarized capacitor"
 			(at 63.5 44.45 0)
 			(effects
@@
 		)
 	)
+	(embedded_fonts no)
 )
